File: brownbox/brownbox.kicad_pcb (KiCad board)
At the start: 2 copper layers, 260 parts, among them J1 Rifle Connector - C7-205, J2 12-Pin Cinch Jones Expansion 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, J3 Jumper, Q1 2N5134, Q10 2N5134, Q11 2N5133, Q12 2N5134, Q13 2N5134, Q14 2N5134, Q15 2N5133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

Commit message: Update to kicad6
Other:
- net class Default removed
