File: brownbox/brownbox.kicad_pcb (KiCad board)
At the start: 2 copper layers, 260 parts, among them J1 Rifle Connector - C7-205, J2 12-Pin Cinch Jones Expansion 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, J3 Jumper, Q1 2N5134, Q10 2N5134, Q11 2N5133, Q12 2N5134, Q13 2N5134, Q14 2N5134, Q15 2N5133, Q16 2N5134, Q17 2N5134, Q18 2N5134, Q19 2N5133, Q2 2N5139, Q20 2N5134, Q21 2N5133, Q22 2N5139, Q23 2N5133, Q24 2N5139, Q25 2N5133, Q26 2N5139, Q27 2N5133, Q28 2N5139, Q29 2N5134, Q3 2N5134, Q30 2N5134, Q31 2N5133, Q32 2N5133, Q33 2N5133, Q34 2N5133, Q35 2N5134, Q36 2N5134, Q37 2N5133, Q38 2N5133, Q39 2N5133, Q4 2N5139, Q40 2N5139, Q41 2N5139, Q42 2N5133, Q43 2N5139, Q44 2N5133, Q45 2N5133, Q46 2N5133, Q5 2N5134, Q6 2N5134, Q7 2N5133, Q8 2N5134, Q9 2N5134

Commit message: capacitor footprints picked and some layout started
Parts:
- added C1: 390pF, Capacitor_THT:C_Disc_D5.0mm_W2.5mm_P5.00mm, F.Cu at (37.5, 54.0)
- added C10: 0.1uF, Capacitor_THT:C_Disc_D5.0mm_W2.5mm_P5.00mm, F.Cu at (-221.2, 53.6)
- added C11: 0.01uF, Capacitor_THT:C_Disc_D5.0mm_W2.5mm_P5.00mm, F.Cu at (-229.3, 61.7)
- added C12: 100uF, Capacitor_THT:C_Disc_D5.0mm_W2.5mm_P5.00mm, F.Cu at (-237.5, 69.8)
- added C13: 100uF, Capacitor_THT:C_Disc_D5.0mm_W2.5mm_P5.00mm, F.Cu at (-237.5, 73.8)
- added C14: 750pF, Capacitor_THT:C_Disc_D5.0mm_W2.5mm_P5.00mm, F.Cu at (-213.0, 49.5)
- added C15: 0.1uF, Capacitor_THT:C_Disc_D5.0mm_W2.5mm_P5.00mm, F.Cu at (-229.3, 65.7)
- added C16: 130pF, Capacitor_THT:C_Disc_D5.0mm_W2.5mm_P5.00mm, F.Cu at (-221.2, 57.6)
- added C17: 0.1uF, Capacitor_THT:C_Disc_D5.0mm_W2.5mm_P5.00mm, F.Cu at (-213.0, 53.6)
- added C18: 0.01uF, Capacitor_THT:C_Disc_D5.0mm_W2.5mm_P5.00mm, F.Cu at (-221.2, 61.7)
- added C19: 100uF, Capacitor_THT:C_Disc_D5.0mm_W2.5mm_P5.00mm, F.Cu at (-237.5, 81.9)
- added C2: 330pF, Capacitor_THT:C_Disc_D5.0mm_W2.5mm_P5.00mm, F.Cu at (57.1, 38.7)
- added C20: 100uF, Capacitor_THT:C_Disc_D5.0mm_W2.5mm_P5.00mm, F.Cu at (-221.2, 65.7)
- added C21: 750pF, Capacitor_THT:C_Disc_D5.0mm_W2.5mm_P5.00mm, F.Cu at (-229.3, 73.8)
- added C22: 0.1uF, Capacitor_THT:C_Disc_D5.0mm_W2.5mm_P5.00mm, F.Cu at (-213.0, 57.6)
- added C23: 130pF, Capacitor_THT:C_Disc_D5.0mm_W2.5mm_P5.00mm, F.Cu at (-204.9, 53.6)
- added C24: 0.1uF, Capacitor_THT:C_Disc_D5.0mm_W2.5mm_P5.00mm, F.Cu at (-213.0, 61.7)
- added C25: 750pF, Capacitor_THT:C_Disc_D5.0mm_W2.5mm_P5.00mm, F.Cu at (-229.3, 69.8)
- added C26: 0.1uF, Capacitor_THT:C_Disc_D5.0mm_W2.5mm_P5.00mm, F.Cu at (-237.5, 77.9)
- added C27: 130pF, Capacitor_THT:C_Disc_D5.0mm_W2.5mm_P5.00mm, F.Cu at (-204.9, 49.5)
- added C28: 0.1uF, Capacitor_THT:C_Disc_D5.0mm_W2.5mm_P5.00mm, F.Cu at (-221.2, 69.8)
- added C29: 0.1uF, Capacitor_THT:C_Disc_D5.0mm_W2.5mm_P5.00mm, F.Cu at (-196.7, 49.5)
- added C3: 0.1uF, Capacitor_THT:C_Disc_D5.0mm_W2.5mm_P5.00mm, F.Cu at (37.5, 88.3)
- added C30: 100pF, Capacitor_THT:C_Disc_D5.0mm_W2.5mm_P5.00mm, F.Cu at (-229.3, 77.9)
- added C31: 100pF, Capacitor_THT:C_Disc_D5.0mm_W2.5mm_P5.00mm, F.Cu at (-229.3, 81.9)
- added C32: 0.1uF, Capacitor_THT:C_Disc_D5.0mm_W2.5mm_P5.00mm, F.Cu at (-213.0, 65.7)
- added C33: 0.1uF, Capacitor_THT:C_Disc_D5.0mm_W2.5mm_P5.00mm, F.Cu at (-196.7, 53.6)
- added C34: 100pF, Capacitor_THT:C_Disc_D5.0mm_W2.5mm_P5.00mm, F.Cu at (-204.9, 57.6)
- added C35: 100pF, Capacitor_THT:C_Disc_D5.0mm_W2.5mm_P5.00mm, F.Cu at (-204.9, 61.7)
- added C36: 82pF, Capacitor_THT:C_Disc_D5.0mm_W2.5mm_P5.00mm, F.Cu at (-213.0, 77.9)
- added C37: 180pF, Capacitor_THT:C_Disc_D5.0mm_W2.5mm_P5.00mm, F.Cu at (-204.9, 69.8)
- added C38: 0.22uF, Capacitor_THT:C_Disc_D5.0mm_W2.5mm_P5.00mm, F.Cu at (-213.0, 69.8)
- added C39: 0.1uF, Capacitor_THT:C_Disc_D5.0mm_W2.5mm_P5.00mm, F.Cu at (-221.2, 77.9)
- added C4: 0.2uF, Capacitor_THT:C_Disc_D5.0mm_W2.5mm_P5.00mm, F.Cu at (57.7, 73.0)
- added C40: 27pF, Capacitor_THT:C_Disc_D5.0mm_W2.5mm_P5.00mm, F.Cu at (-196.7, 69.8)
- added C41: 0.01uF, Capacitor_THT:C_Disc_D5.0mm_W2.5mm_P5.00mm, F.Cu at (-188.6, 57.6)
- added C42: 62pF, Capacitor_THT:C_Disc_D5.0mm_W2.5mm_P5.00mm, F.Cu at (-213.0, 81.9)
- added C43: 180pF, Capacitor_THT:C_Disc_D5.0mm_W2.5mm_P5.00mm, F.Cu at (-196.7, 65.7)
- added C44: 56pF, Capacitor_THT:C_Disc_D5.0mm_W2.5mm_P5.00mm, F.Cu at (-204.9, 73.8)
- added C45: 360pF, Capacitor_THT:C_Disc_D5.0mm_W2.5mm_P5.00mm, F.Cu at (-188.6, 61.7)
- added C46: 120pF, Capacitor_THT:C_Disc_D5.0mm_W2.5mm_P5.00mm, F.Cu at (-180.4, 53.6)
- added C47: 0.1uF, Capacitor_THT:C_Disc_D5.0mm_W2.5mm_P5.00mm, F.Cu at (-196.7, 57.6)
- added C48: 0.01uF, Capacitor_THT:C_Disc_D5.0mm_W2.5mm_P5.00mm, F.Cu at (-213.0, 73.8)
- added C49: 0.01uF, Capacitor_THT:C_Disc_D5.0mm_W2.5mm_P5.00mm, F.Cu at (-204.9, 65.7)
- added C5: 100uF, Capacitor_THT:C_Disc_D5.0mm_W2.5mm_P5.00mm, F.Cu at (-229.3, 53.6)
- added C50: 0.01uF, Capacitor_THT:C_Disc_D5.0mm_W2.5mm_P5.00mm, F.Cu at (-188.6, 53.6)
- added C51: 0.3uF, Capacitor_THT:C_Disc_D5.0mm_W2.5mm_P5.00mm, F.Cu at (-188.6, 49.5)
- added C52: 0.1uF, Capacitor_THT:C_Disc_D5.0mm_W2.5mm_P5.00mm, F.Cu at (-196.7, 61.7)
- added C53: 0.1uF, Capacitor_THT:C_Disc_D5.0mm_W2.5mm_P5.00mm, F.Cu at (-221.2, 81.9)
- added C54: 10uF, Capacitor_THT:C_Disc_D5.0mm_W2.5mm_P5.00mm, F.Cu at (-204.9, 77.9)
- added C55: 10uF, Capacitor_THT:C_Disc_D5.0mm_W2.5mm_P5.00mm, F.Cu at (-204.9, 81.9)
- added C56: 0.02uF, Capacitor_THT:C_Disc_D5.0mm_W2.5mm_P5.00mm, F.Cu at (-196.7, 73.8)
- added C6: 100uF, Capacitor_THT:C_Disc_D5.0mm_W2.5mm_P5.00mm, F.Cu at (-221.2, 49.5)
- added C7: 750pF, Capacitor_THT:C_Disc_D5.0mm_W2.5mm_P5.00mm, F.Cu at (-237.5, 61.7)
- added C8: 0.1uF, Capacitor_THT:C_Disc_D5.0mm_W2.5mm_P5.00mm, F.Cu at (-237.5, 65.7)
- added C9: 130pF, Capacitor_THT:C_Disc_D5.0mm_W2.5mm_P5.00mm, F.Cu at (-229.3, 57.6)
- added CV1: 9-35pF, Capacitor_THT:C_Disc_D5.0mm_W2.5mm_P5.00mm, F.Cu at (-221.2, 73.8)
- added CV2: 9-35pF, Capacitor_THT:C_Disc_D5.0mm_W2.5mm_P5.00mm, F.Cu at (-180.4, 49.5)
- moved BT1 292.2 mm to (-88.6, 104.8)
- moved BT2 292.2 mm to (-114.9, 128.6)
- moved D1 292.2 mm to (-217.2, 141.1)
- moved D10 292.2 mm to (-163.4, 136.7)
- moved D12 292.2 mm to (-143.2, 112.4)
- moved D13 292.2 mm to (-196.9, 168.4)
- moved D14 292.2 mm to (-218.4, 189.0)
- moved D15 292.2 mm to (-207.7, 184.6)
- moved D16 292.2 mm to (-144.9, 120.0)
- moved D18 292.2 mm to (-186.1, 187.2)
- moved D19 292.2 mm to (-100.1, 104.3)
- moved D2 292.2 mm to (-197.0, 115.9)
- moved D21 292.2 mm to (-110.8, 112.4)
- moved D22 292.2 mm to (-164.6, 166.6)
- moved D24 292.2 mm to (-152.6, 132.6)
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Other:
- board text added: "Horiz. Sync Multivibrator"
- board text added: "Vert. Sync Multivibrator"

Commit message: more layout
Parts:
- moved C1 22.5 mm to (26.7, 34.3)
- moved C3 22.5 mm to (26.7, 68.6)
- moved Q2 22.5 mm to (53.0, 17.8)
- moved Q3 22.5 mm to (17.1, 69.8)
- moved R1 22.5 mm to (17.1, 24.8)
- moved R11 22.5 mm to (23.5, 60.3)
- moved R2 22.5 mm to (41.3, 24.8)
- moved R3 22.5 mm to (41.9, 34.3)
- moved R4 22.5 mm to (53.3, 29.2)
- moved R6 22.5 mm to (46.4, 29.2)
- moved R9 22.5 mm to (41.9, 68.6)
- moved RV2 22.5 mm to (23.5, 51.5)
- moved C2 22.5 mm to (46.3, 19.1)
- moved C4 22.5 mm to (47.0, 53.3)
- moved Q1 22.5 mm to (17.1, 35.6)
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Changed lines of the file:
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@@
   )
   (footprint "Resistor_THT:R_Axial_DIN0207_L6.3mm_D2.5mm_P7.62mm_Horizontal" (layer "F.Cu")
-    (at 27.94 44.45 90)
+    (at 17.145 24.765 90)
     (descr "Resistor, Axial_DIN0207 series, Axial, Horizontal, pin pitch=7.62mm, 0.25W = 1/4W, length*diameter=6.3*2.5mm^2, http://cdn-reichelt.de/documents/datenblatt/B400/1_4W%23YAG.pdf")
     (tags "Resistor Axial_DIN0207 series Axial Horizontal pin pitch 7.62mm 0.25W = 1/4W length 6.3mm diameter 2.5mm")
@@
   )
   (footprint "Resistor_THT:R_Axial_DIN0207_L6.3mm_D2.5mm_P7.62mm_Horizontal" (layer "F.Cu")
-    (at 27.94 78.74 90)
+    (at 17.145 59.055 90)
     (descr "Resistor, Axial_DIN0207 series, Axial, Horizontal, pin pitch=7.62mm, 0.25W = 1/4W, length*diameter=6.3*2.5mm^2, http://cdn-reichelt.de/documents/datenblatt/B400/1_4W%23YAG.pdf")
     (tags "Resistor Axial_DIN0207 series Axial Horizontal pin pitch 7.62mm 0.25W = 1/4W length 6.3mm diameter 2.5mm")
@@
   )
   (footprint "Resistor_THT:R_Axial_DIN0207_L6.3mm_D2.5mm_P7.62mm_Horizontal" (layer "F.Cu")
-    (at 64.135 48.895 -90)
+    (at 53.34 29.21 -90)
     (descr "Resistor, Axial_DIN0207 series, Axial, Horizontal, pin pitch=7.62mm, 0.25W = 1/4W, length*diameter=6.3*2.5mm^2, http://cdn-reichelt.de/documents/datenblatt/B400/1_4W%23YAG.pdf")
     (tags "Resistor Axial_DIN0207 series Axial Horizontal pin pitch 7.62mm 0.25W = 1/4W length 6.3mm diameter 2.5mm")
@@
   )
   (footprint "Capacitor_THT:C_Disc_D5.0mm_W2.5mm_P5.00mm" (layer "F.Cu")
-    (at 57.11 38.735 180)
+    (at 46.315 19.05 180)
     (descr "C, Disc series, Radial, pin pitch=5.00mm, , diameter*width=5*2.5mm^2, Capacitor, http://cdn-reichelt.de/documents/datenblatt/B300/DS_KERKO_TC.pdf")
     (tags "C Disc series Radial pin pitch 5.00mm  diameter 5mm width 2.5mm Capacitor")
@@
   )
   (footprint "Resistor_THT:R_Axial_DIN0207_L6.3mm_D2.5mm_P7.62mm_Horizontal" (layer "F.Cu")
-    (at 34.29 80.01 -90)
+    (at 23.495 60.325 -90)
     (descr "Resistor, Axial_DIN0207 series, Axial, Horizontal, pin pitch=7.62mm, 0.25W = 1/4W, length*diameter=6.3*2.5mm^2, http://cdn-reichelt.de/documents/datenblatt/B400/1_4W%23YAG.pdf")
     (tags "Resistor Axial_DIN0207 series Axial Horizontal pin pitch 7.62mm 0.25W = 1/4W length 6.3mm diameter 2.5mm")
@@
   )
   (footprint "Resistor_THT:R_Axial_DIN0207_L6.3mm_D2.5mm_P7.62mm_Horizontal" (layer "F.Cu")
-    (at 52.705 53.975 180)
+    (at 41.91 34.29 180)
     (descr "Resistor, Axial_DIN0207 series, Axial, Horizontal, pin pitch=7.62mm, 0.25W = 1/4W, length*diameter=6.3*2.5mm^2, http://cdn-reichelt.de/documents/datenblatt/B400/1_4W%23YAG.pdf")
     (tags "Resistor Axial_DIN0207 series Axial Horizontal pin pitch 7.62mm 0.25W = 1/4W length 6.3mm diameter 2.5mm")
@@
   )
   (footprint "Potentiometer_THT:Potentiometer_Bourns_3266W_Vertical" (layer "F.Cu")
-    (at 34.335 71.135 90)
+    (at 23.54 51.45 90)
     (descr "Potentiometer, vertical, Bourns 3266W, https://www.bourns.com/docs/Product-Datasheets/3266.pdf")
     (tags "Potentiometer vertical Bourns 3266W")
@@
   )
   (footprint "Resistor_THT:R_Axial_DIN0207_L6.3mm_D2.5mm_P7.62mm_Horizontal" (layer "F.Cu")
-    (at 34.29 45.72 -90)
+    (at 23.495 26.035 -90)
     (descr "Resistor, Axial_DIN0207 series, Axial, Horizontal, pin pitch=7.62mm, 0.25W = 1/4W, length*diameter=6.3*2.5mm^2, http://cdn-reichelt.de/documents/datenblatt/B400/1_4W%23YAG.pdf")
     (tags "Resistor Axial_DIN0207 series Axial Horizontal pin pitch 7.62mm 0.25W = 1/4W length 6.3mm diameter 2.5mm")
@@
   )
   (footprint "Potentiometer_THT:Potentiometer_Bourns_3266W_Vertical" (layer "F.Cu")
-    (at 34.335 36.845 90)
+    (at 23.54 17.16 90)
     (descr "Potentiometer, vertical, Bourns 3266W, https://www.bourns.com/docs/Product-Datasheets/3266.pdf")
     (tags "Potentiometer vertical Bourns 3266W")
@@
   )
   (footprint "footprints:TO-92_Offset_TO-106" (layer "F.Cu")
-    (at 64.135 71.755 -90)
+    (at 53.34 52.07 -90)
     (descr "TO-92 leads compatable with TO-106, narrow, oval pads, drill 0.75mm (see NXP sot054_po.pdf)")
     (tags "to-92 sc-43 sc-43a sot54 PA33 transistor")
@@
   )
   (footprint "Capacitor_THT:C_Disc_D5.0mm_W2.5mm_P5.00mm" (layer "F.Cu")
-    (at 57.745 73.025 180)
+    (at 46.95 53.34 180)
     (descr "C, Disc series, Radial, pin pitch=5.00mm, , diameter*width=5*2.5mm^2, Capacitor, http://cdn-reichelt.de/documents/datenblatt/B300/DS_KERKO_TC.pdf")
     (tags "C Disc series Radial pin pitch 5.00mm  diameter 5mm width 2.5mm Capacitor")
@@
   )
   (footprint "Resistor_THT:R_Axial_DIN0207_L6.3mm_D2.5mm_P7.62mm_Horizontal" (layer "F.Cu")
-    (at 57.785 80.645 -90)
+    (at 46.99 60.96 -90)
     (descr "Resistor, Axial_DIN0207 series, Axial, Horizontal, pin pitch=7.62mm, 0.25W = 1/4W, length*diameter=6.3*2.5mm^2, http://cdn-reichelt.de/documents/datenblatt/B400/1_4W%23YAG.pdf")
     (tags "Resistor Axial_DIN0207 series Axial Horizontal pin pitch 7.62mm 0.25W = 1/4W length 6.3mm diameter 2.5mm")
@@
   )
   (footprint "Resistor_THT:R_Axial_DIN0207_L6.3mm_D2.5mm_P7.62mm_Horizontal" (layer "F.Cu")
-    (at 52.705 88.265 180)
+    (at 41.91 68.58 180)
     (descr "Resistor, Axial_DIN0207 series, Axial, Horizontal, pin pitch=7.62mm, 0.25W = 1/4W, length*diameter=6.3*2.5mm^2, http://cdn-reichelt.de/documents/datenblatt/B400/1_4W%23YAG.pdf")
     (tags "Resistor Axial_DIN0207 series Axial Horizontal pin pitch 7.62mm 0.25W = 1/4W length 6.3mm diameter 2.5mm")
@@
   )
   (footprint "Resistor_THT:R_Axial_DIN0207_L6.3mm_D2.5mm_P7.62mm_Horizontal" (layer "F.Cu")
-    (at 52.07 44.45 180)
+    (at 41.275 24.765 180)
     (descr "Resistor, Axial_DIN0207 series, Axial, Horizontal, pin pitch=7.62mm, 0.25W = 1/4W, length*diameter=6.3*2.5mm^2, http://cdn-reichelt.de/documents/datenblatt/B400/1_4W%23YAG.pdf")
     (tags "Resistor Axial_DIN0207 series Axial Horizontal pin pitch 7.62mm 0.25W = 1/4W length 6.3mm diameter 2.5mm")
@@
   )
   (footprint "Resistor_THT:R_Axial_DIN0207_L6.3mm_D2.5mm_P7.62mm_Horizontal" (layer "F.Cu")
-    (at 57.15 48.895 -90)
+    (at 46.355 29.21 -90)
     (descr "Resistor, Axial_DIN0207 series, Axial, Horizontal, pin pitch=7.62mm, 0.25W = 1/4W, length*diameter=6.3*2.5mm^2, http://cdn-reichelt.de/documents/datenblatt/B400/1_4W%23YAG.pdf")
     (tags "Resistor Axial_DIN0207 series Axial Horizontal pin pitch 7.62mm 0.25W = 1/4W length 6.3mm diameter 2.5mm")
@@
   )
   (footprint "footprints:TO-92_Offset_TO-106" (layer "F.Cu")
-    (at 27.94 89.535 90)
+    (at 17.145 69.85 90)
     (descr "TO-92 leads compatable with TO-106, narrow, oval pads, drill 0.75mm (see NXP sot054_po.pdf)")
     (tags "to-92 sc-43 sc-43a sot54 PA33 transistor")
@@
   )
   (footprint "footprints:TO-92_Offset_TO-106" (layer "F.Cu")
-    (at 27.94 55.245 90)
+    (at 17.145 35.56 90)
     (descr "TO-92 leads compatable with TO-106, narrow, oval pads, drill 0.75mm (see NXP sot054_po.pdf)")
     (tags "to-92 sc-43 sc-43a sot54 PA33 transistor")
@@
   )
   (footprint "Capacitor_THT:C_Disc_D5.0mm_W2.5mm_P5.00mm" (layer "F.Cu")
-    (at 37.505 88.265)
+    (at 26.71 68.58)
     (descr "C, Disc series, Radial, pin pitch=5.00mm, , diameter*width=5*2.5mm^2, Capacitor, http://cdn-reichelt.de/documents/datenblatt/B300/DS_KERKO_TC.pdf")
     (tags "C Disc series Radial pin pitch 5.00mm  diameter 5mm width 2.5mm Capacitor")
@@
   )
   (footprint "footprints:TO-92_Offset_TO-106" (layer "F.Cu")
-    (at 63.775 37.465 -90)
+    (at 52.98 17.78 -90)
     (descr "TO-92 leads compatable with TO-106, narrow, oval pads, drill 0.75mm (see NXP sot054_po.pdf)")
     (tags "to-92 sc-43 sc-43a sot54 PA33 transistor")
@@
   )
   (footprint "Resistor_THT:R_Axial_DIN0207_L6.3mm_D2.5mm_P7.62mm_Horizontal" (layer "F.Cu")
-    (at 64.77 80.645 -90)
+    (at 53.975 60.96 -90)
     (descr "Resistor, Axial_DIN0207 series, Axial, Horizontal, pin pitch=7.62mm, 0.25W = 1/4W, length*diameter=6.3*2.5mm^2, http://cdn-reichelt.de/documents/datenblatt/B400/1_4W%23YAG.pdf")
     (tags "Resistor Axial_DIN0207 series Axial Horizontal pin pitch 7.62mm 0.25W = 1/4W length 6.3mm diameter 2.5mm")
@@
   )
   (footprint "Capacitor_THT:C_Disc_D5.0mm_W2.5mm_P5.00mm" (layer "F.Cu")
-    (at 37.465 53.975)
+    (at 26.67 34.29)
     (descr "C, Disc series, Radial, pin pitch=5.00mm, , diameter*width=5*2.5mm^2, Capacitor, http://cdn-reichelt.de/documents/datenblatt/B300/DS_KERKO_TC.pdf")
     (tags "C Disc series Radial pin pitch 5.00mm  diameter 5mm width 2.5mm Capacitor")
@@
   )
   (footprint "Resistor_THT:R_Axial_DIN0207_L6.3mm_D2.5mm_P7.62mm_Horizontal" (layer "F.Cu")
-    (at 52.705 78.74 180)
+    (at 41.91 59.055 180)
     (descr "Resistor, Axial_DIN0207 series, Axial, Horizontal, pin pitch=7.62mm, 0.25W = 1/4W, length*diameter=6.3*2.5mm^2, http://cdn-reichelt.de/documents/datenblatt/B400/1_4W%23YAG.pdf")
     (tags "Resistor Axial_DIN0207 series Axial Horizontal pin pitch 7.62mm 0.25W = 1/4W length 6.3mm diameter 2.5mm")
@@
     )
   )
-  (gr_text "Horiz. Sync Multivibrator" (at 45.085 33.655) (layer "F.SilkS")
+  (gr_text "Horiz. Sync Multivibrator" (at 34.29 13.97) (layer "F.SilkS")
     (effects (font (size 1 1) (thickness 0.15)))
   )
-  (gr_text "Vert. Sync Multivibrator" (at 45.085 67.945) (layer "F.SilkS")
+  (gr_text "Vert. Sync Multivibrator" (at 34.29 48.26) (layer "F.SilkS")
     (effects (font (size 1 1) (thickness 0.15)))
   )

Commit message: more preliminary layout
Parts:
- moved R91 417.3 mm to (20.7, -152.4)
- moved R113 382.2 mm to (50.1, -99.7), turned to -90 degrees
- moved R93 379.5 mm to (13.1, -127.6)
- moved R114 377.3 mm to (62.2, -86.4), turned to -90 degrees
- moved Q32 375.8 mm to (31.5, -126.4), turned to 90 degrees
- moved R115 370.2 mm to (93.3, -86.4), turned to -90 degrees
- moved R89 366.6 mm to (31.5, -160.0), turned to -90 degrees
- moved R90 354.1 mm to (31.5, -140.3), turned to -90 degrees
- moved D37 352.7 mm to (78.7, -53.3), turned to -90 degrees
- moved Q37 350.3 mm to (32.3, -87.6), turned to 90 degrees
- moved R92 347.6 mm to (20.7, -132.7)
- moved D31 337.6 mm to (17.7, -59.1)
- moved R120 337.3 mm to (81.9, -45.7)
- moved R131 332.7 mm to (74.9, -30.5), turned to 180 degrees
- moved R94 323.4 mm to (20.7, -124.5), turned to -90 degrees
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Other:
- board text added: "Joystick Amps"
- board text added: "Odd/Evan Code Gen"

Commit message: still working on placement
Parts:
- moved R88 354.1 mm to (121.9, -15.9)
- moved R24 329.2 mm to (100.3, 84.5), turned to -90 degrees
- moved C9 305.3 mm to (73.7, 95.2)
- moved R21 294.3 mm to (83.2, 84.5), turned to -90 degrees
- moved R23 290.4 mm to (88.3, 84.5)
- moved C7 285.3 mm to (45.7, 96.5)
- moved R15 278.9 mm to (40.6, 99.7), turned to -90 degrees
- moved C5 276.9 mm to (40.6, 115.0), turned to -90 degrees
- moved D1 256.7 mm to (35.6, 96.5), turned to 180 degrees
- moved R13 249.2 mm to (27.9, 111.1)
- moved R19 243.3 mm to (66.7, 84.5), turned to -90 degrees
- moved R17 242.9 mm to (55.9, 84.5), turned to -90 degrees
- moved Q6 241.1 mm to (100.3, 97.8), turned to 90 degrees
- moved C37 221.5 mm to (128.3, -43.2)
- moved R86 221.1 mm to (145.4, -43.2), turned to 90 degrees
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
Commit message: finished initial placement
Parts:
- added X1: 3.579545Mhz, Crystal:Crystal_HC49-U_Horizontal, F.Cu at (268.0, -243.1)
- moved R98 694.8 mm to (358.8, -189.9)
- moved R108 685.3 mm to (370.2, -261.0)
- moved R107 684.8 mm to (341.6, -262.3), turned to -90 degrees
- moved R109 683.7 mm to (357.5, -253.4), turned to 90 degrees
- moved R106 676.2 mm to (328.3, -262.3)
- moved D28 664.5 mm to (335.9, -254.6), turned to 180 degrees
- moved R96 657.1 mm to (343.5, -197.5), turned to -90 degrees
- moved RV9 656.0 mm to (320.0, -251.5), turned to 90 degrees
- moved R97 654.9 mm to (372.7, -197.5), turned to -90 degrees
- moved R99 653.7 mm to (335.9, -174.6), turned to -90 degrees
- moved J2 643.5 mm to (355.5, -144.1)
- moved R146 643.2 mm to (335.9, -113.7), turned to -90 degrees
- moved J1 639.5 mm to (357.4, -104.1)
- moved C45 637.8 mm to (364.5, -256.0), turned to 90 degrees
- moved R101 636.8 mm to (377.2, -156.2), turned to 90 degrees
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Other:
- board text added: "chroma gen"
- board text added: "primary flip flop"
- board text added: "secondary flip flop"
- board text added: "spot gen, ball"
- board text added: "spot gen, left"
- board text added: "spot gen, net"
- board text added: "spot gen, right"
